File: hardware/dash.kicad_sch (KiCad schematic)
At the start: 20 parts, among them J1 Conn_01x26, Q1 Si1308EDL, U1 SCD40-D-R2

Commit message: update schema
Parts:
- added C11: 4.7u, symbol Device:C_Small
- added C12: 47u, symbol Device:C_Small
- added C13, C14: 0.1u, symbol Device:C_Small
- added L2: L_Ferrite, symbol Device:L_Ferrite
- added R3, R4: 10k, symbol Device:R
- C10: value 4.7u -> 47u; symbol Device:C -> Device:C_Small
Connections:
- net +3.3V: now also U1.19 (VDD), U1.7 (VDD), C12.1, C13.1, L2.1, R3.1, R4.1; no longer C10.1, L1.1
- net GND: now also J1.25 (MP), J1.26 (MP), U1.20 (GND), U1.21 (GND), U1.6 (GND), C11.2, C12.2, C13.2, C14.2
- net SCL: now also U1.9 (SCL), R4.2
- net SDA: now also U1.10 (SDA), R3.2
- new net: C10.1, C11.1, C14.1, L1.1, L2.2
Other:
- moved on the sheet: C10, Q1, R1, R2

Commit message: schmatic complete
Parts:
- removed A1: RaspberryPi_Pico_W, Module:RaspberryPi_Pico_W_SMD_HandSolder, symbol MCU_Module:RaspberryPi_Pico_W
- added U2: M5Stamp-C3, My_lib:M5Stamp_C3, symbol My_lib:M5Stamp_C3
- C1, C13, C14, C2, C3, C4, C5, C6, C7, C8: footprint (none) -> Capacitor_SMD:C_0603_1608Metric_Pad1.08x0.95mm_HandSolder
- C10, C11, C12, C9: footprint (none) -> Capacitor_SMD:C_0805_2012Metric_Pad1.18x1.45mm_HandSolder
- D1, D2, D3: value MBR0530 -> D_Schottky; footprint Diode_SMD:D_SOD-123 -> Diode_SMD:D_SMA; symbol Diode:MBR0530 -> Device:D_Schottky
- J1: value Conn_01x26 -> Conn_Display; footprint (none) -> Connector_FFC-FPC:Jushuo_AFC07-S24FCA-00_1x24-1MP_P0.50_Horizontal
- L1: footprint (none) -> Inductor_SMD:L_10.4x10.4_H4.8
- L2: footprint (none) -> Inductor_SMD:L_0603_1608Metric_Pad1.05x0.95mm_HandSolder
- Q1: value Si1308EDL -> AO3400A; footprint Package_TO_SOT_SMD:SOT-323_SC-70 -> Package_TO_SOT_SMD:SOT-23_Handsoldering; symbol Transistor_FET:Si1308EDL -> Transistor_FET:AO3400A
- R1: value 1M -> 10k; footprint (none) -> Resistor_SMD:R_0603_1608Metric_Pad0.98x0.95mm_HandSolder
- R2, R3, R4: footprint (none) -> Resistor_SMD:R_0603_1608Metric_Pad0.98x0.95mm_HandSolder
Connections:
- net +3.3V: now also U2.22 (3V3)
- net BUSY: now also U2.7 (G10)
- net GND: now also J1.MP, U2.1 (GND), U2.13 (GND), U2.17 (GND), U2.9 (GND); no longer J1.25 (MP), J1.26 (MP)
- net SCL: now also U2.12 (G0); no longer J1.13 (SCL)
- net SDA: now also U2.11 (G1); no longer J1.14 (SDA)
- net ~{CS}: now also U2.3 (G5)
- net ~{D/C}: now also U2.2 (G4)
- net ~{RES}: now also U2.6 (G8)
- new net MOSI: J1.14 (SDA), U2.5 (G7)
- new net SCK: J1.13 (SCL), U2.4 (G6)
- no-connect marks 3 -> 14
Other:
- moved on the sheet: C1, C10, C11, C12, C13, C14, C2, C3, C4, C5, C6, C7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

Commit message: finish pcb
Parts:
- renumbered U2 to U1, U1 to U2
Changed lines of the file:
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@@
 		(dnp no)
 		(fields_autoplaced yes)
-		(property "Reference" "U1"
+		(property "Reference" "U2"
 			(at 36.83 41.9099 0)
 			(effects
@@
 			(project ""
 				(path "/fb40bc52-0d55-4a87-be84-6a78ea7f72ee"
-					(reference "U1")
+					(reference "U2")
 					(unit 1)
 				)
@@
 		(dnp no)
 		(fields_autoplaced yes)
-		(property "Reference" "U2"
+		(property "Reference" "U1"
 			(at 231.14 33.02 0)
 			(effects
@@
 			(project ""
 				(path "/fb40bc52-0d55-4a87-be84-6a78ea7f72ee"
-					(reference "U2")
-					(unit 1)
-				)
+					(reference "U1")
+					(unit 1)
+				)
