File: hardware/dash.kicad_pcb (KiCad board)
At the start: 2 copper layers, 100 x 36.7 mm, 28 parts, among them J1 Conn_Display, Q1 AO3400A, U1 M5Stamp-C3, U2 SCD40-D-R2

Commit message: fix
Routing:
- net +3.3V: track 116.0 -> 145.7 mm
- net GND: track 270.5 -> 272.6 mm, vias 30 -> 31
